File: TeaCup(C)3.3/12-30-23-Teacup.kicad_pcb-revC.kicad_sch (KiCad schematic)
At the start: 107 parts, among them IC1 T31ZX, J1 USB Type-C, J10 AudioJack4_Ground, J11 Conn_01x04_Pin, J12 Conn_01x04_Pin, J13 SFW15R-2STE1LF, J14 Conn_01x02_MountingPin, J15 Conn_01x03_MountingPin, J16 Conn_01x03_MountingPin, J2 Micro_SD_Card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

Commit message: update silk
Parts:
- removed LOGO3, LOGO4: Teacup Logo, Symbol:Symbol_GNU-Logo_SilkscreenTop, symbol Graphic:Logo_Open_Hardware_Small
- LOGO2: value Teacup Logo -> OSHW OUTLINE; footprint Symbol:OSHW-Logo_19x20mm_SilkScreen -> teacup:oshw
- LOGO5: value Teacup Logo -> OSHW SMALL
Changed lines of the file:
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@@
     )
   )
-  (symbol (lib_id "Graphic:Logo_Open_Hardware_Small") (at 291.973 97.917 0) (unit 1)
+  (symbol (lib_id "Graphic:Logo_Open_Hardware_Small") (at 312.674 101.473 0) (unit 1)
     (in_bom no) (on_board yes) (dnp no) (fields_autoplaced)
-    (property "Reference" "LOGO5" (at 291.973 90.932 0)
+    (property "Reference" "LOGO5" (at 312.674 94.488 0)
       (effects (font (size 1.27 1.27)) hide)
     )
-    (property "Value" "Teacup Logo" (at 298.45 97.917 0)
+    (property "Value" "OSHW SMALL" (at 319.151 101.473 0)
       (effects (font (size 1.27 1.27)) (justify left))
     )
-    (property "Footprint" "Symbol:OSHW-Logo_7.5x8mm_SilkScreen" (at 291.973 97.917 0)
+    (property "Footprint" "Symbol:OSHW-Logo_7.5x8mm_SilkScreen" (at 312.674 101.473 0)
       (effects (font (size 1.27 1.27)) hide)
     )
-    (property "Datasheet" "~" (at 291.973 97.917 0)
+    (property "Datasheet" "~" (at 312.674 101.473 0)
       (effects (font (size 1.27 1.27)) hide)
     )
-    (property "Sim.Enable" "0" (at 291.973 97.917 0)
+    (property "Sim.Enable" "0" (at 312.674 101.473 0)
       (effects (font (size 1.27 1.27)) hide)
     )
@@
     )
   )
-  (symbol (lib_id "Graphic:Logo_Open_Hardware_Small") (at 391.16 99.06 0) (unit 1)
+  (symbol (lib_id "Graphic:Logo_Open_Hardware_Small") (at 312.42 110.744 0) (unit 1)
     (in_bom no) (on_board yes) (dnp no) (fields_autoplaced)
-    (property "Reference" "LOGO1" (at 391.16 92.075 0)
+    (property "Reference" "LOGO1" (at 312.42 103.759 0)
       (effects (font (size 1.27 1.27)) hide)
     )
-    (property "Value" "Teacup Logo" (at 391.16 104.775 0)
+    (property "Value" "Teacup Logo" (at 312.42 116.459 0)
       (effects (font (size 1.27 1.27)))
     )
-    (property "Footprint" "teacup:Teacup-logo" (at 391.16 99.06 0)
+    (property "Footprint" "teacup:Teacup-logo" (at 312.42 110.744 0)
       (effects (font (size 1.27 1.27)) hide)
     )
-    (property "Datasheet" "~" (at 391.16 99.06 0)
+    (property "Datasheet" "~" (at 312.42 110.744 0)
       (effects (font (size 1.27 1.27)) hide)
     )
-    (property "Sim.Enable" "0" (at 391.16 99.06 0)
+    (property "Sim.Enable" "0" (at 312.42 110.744 0)
       (effects (font (size 1.27 1.27)) hide)
     )
@@
       (effects (font (size 1.27 1.27)) hide)
     )
-    (property "Value" "Teacup Logo" (at 320.04 92.329 0)
+    (property "Value" "OSHW OUTLINE" (at 320.04 92.329 0)
       (effects (font (size 1.27 1.27)) (justify left))
     )
-    (property "Footprint" "Symbol:OSHW-Logo_19x20mm_SilkScreen" (at 312.674 92.329 0)
+    (property "Footprint" "teacup:oshw" (at 312.674 92.329 0)
       (effects (font (size 1.27 1.27)) hide)
     )
@@
     )
   )
-  (symbol (lib_id "Graphic:Logo_Open_Hardware_Small") (at 298.831 111.379 0) (unit 1)
-    (in_bom no) (on_board yes) (dnp no) (fields_autoplaced)
-    (property "Reference" "LOGO4" (at 298.831 104.394 0)
-      (effects (font (size 1.27 1.27)) hide)
-    )
-    (property "Value" "Teacup Logo" (at 305.943 111.379 0)
-      (effects (font (size 1.27 1.27)) (justify left))
-    )
-    (property "Footprint" "Symbol:Symbol_GNU-Logo_SilkscreenTop" (at 298.831 111.379 0)
-      (effects (font (size 1.27 1.27)) hide)
-    )
-    (property "Datasheet" "~" (at 298.831 111.379 0)
-      (effects (font (size 1.27 1.27)) hide)
-    )
-    (property "Sim.Enable" "0" (at 298.831 111.379 0)
-      (effects (font (size 1.27 1.27)) hide)
-    )
-    (instances
-      (project "12-30-23-Teacup.kicad_pcb-revC"
-        (path "/6e7ef4e6-2026-4726-8de0-60238113f775"
-          (reference "LOGO4") (unit 1)
-        )
-      )
-    )
-  )
   (symbol (lib_id "Device:C") (at 323.85 48.26 0) (unit 1)
     (in_bom yes) (on_board yes) (dnp no) (fields_autoplaced)
@@
         )
       )
-    )
-  )
-  (symbol (lib_id "Graphic:Logo_Open_Hardware_Small") (at 312.928 105.029 0) (unit 1)
-    (in_bom no) (on_board yes) (dnp no) (fields_autoplaced)
-    (property "Reference" "LOGO3" (at 312.928 98.044 0)
-      (effects (font (size 1.27 1.27)) hide)
-    )
-    (property "Value" "Teacup Logo" (at 320.04 105.029 0)
-      (effects (font (size 1.27 1.27)) (justify left))
-    )
-    (property "Footprint" "Symbol:Symbol_GNU-Logo_SilkscreenTop" (at 312.928 105.029 0)
-      (effects (font (size 1.27 1.27)) hide)
-    )
-    (property "Datasheet" "~" (at 312.928 105.029 0)
-      (effects (font (size 1.27 1.27)) hide)
-    )
-    (property "Sim.Enable" "0" (at 312.928 105.029 0)
-      (effects (font (size 1.27 1.27)) hide)
-    )
-    (instances
-      (project "12-30-23-Teacup.kicad_pcb-revC"
-        (path "/6e7ef4e6-2026-4726-8de0-60238113f775"
-          (reference "LOGO3") (unit 1)
-        )
-      )

Commit message: Adjust silk
Parts:
- removed LOGO1: Teacup Logo, teacup:Teacup-logo, symbol Graphic:Logo_Open_Hardware_Small
- removed LOGO5: OSHW SMALL, Symbol:OSHW-Logo_7.5x8mm_SilkScreen, symbol Graphic:Logo_Open_Hardware_Small
- added LOGO3: Teacup Logo, teacup:TClogo-med, symbol Graphic:Logo_Open_Hardware_Small
Changed lines of the file:
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@@
     )
   )
-  (symbol (lib_id "Graphic:Logo_Open_Hardware_Small") (at 312.674 101.473 0) (unit 1)
-    (in_bom no) (on_board yes) (dnp no) (fields_autoplaced)
-    (property "Reference" "LOGO5" (at 312.674 94.488 0)
-      (effects (font (size 1.27 1.27)) hide)
-    )
-    (property "Value" "OSHW SMALL" (at 319.151 101.473 0)
-      (effects (font (size 1.27 1.27)) (justify left))
-    )
-    (property "Footprint" "Symbol:OSHW-Logo_7.5x8mm_SilkScreen" (at 312.674 101.473 0)
-      (effects (font (size 1.27 1.27)) hide)
-    )
-    (property "Datasheet" "~" (at 312.674 101.473 0)
-      (effects (font (size 1.27 1.27)) hide)
-    )
-    (property "Sim.Enable" "0" (at 312.674 101.473 0)
-      (effects (font (size 1.27 1.27)) hide)
-    )
-    (instances
-      (project "12-30-23-Teacup.kicad_pcb-revC"
-        (path "/6e7ef4e6-2026-4726-8de0-60238113f775"
-          (reference "LOGO5") (unit 1)
-        )
-      )
-    )
-  )
   (symbol (lib_id "power:GND") (at 297.18 30.48 0) (unit 1)
     (in_bom yes) (on_board yes) (dnp no)
@@
     )
   )
-  (symbol (lib_id "Graphic:Logo_Open_Hardware_Small") (at 312.42 110.744 0) (unit 1)
-    (in_bom no) (on_board yes) (dnp no) (fields_autoplaced)
-    (property "Reference" "LOGO1" (at 312.42 103.759 0)
-      (effects (font (size 1.27 1.27)) hide)
-    )
-    (property "Value" "Teacup Logo" (at 312.42 116.459 0)
-      (effects (font (size 1.27 1.27)))
-    )
-    (property "Footprint" "teacup:Teacup-logo" (at 312.42 110.744 0)
-      (effects (font (size 1.27 1.27)) hide)
-    )
-    (property "Datasheet" "~" (at 312.42 110.744 0)
-      (effects (font (size 1.27 1.27)) hide)
-    )
-    (property "Sim.Enable" "0" (at 312.42 110.744 0)
-      (effects (font (size 1.27 1.27)) hide)
-    )
-    (instances
-      (project "12-30-23-Teacup.kicad_pcb-revC"
-        (path "/6e7ef4e6-2026-4726-8de0-60238113f775"
-          (reference "LOGO1") (unit 1)
-        )
-      )
-    )
-  )
   (symbol (lib_id "power:GND") (at 78.105 259.08 0) (mirror x) (unit 1)
     (in_bom yes) (on_board yes) (dnp no)
@@
         )
       )
+    )
+  )
+  (symbol (lib_id "Graphic:Logo_Open_Hardware_Small") (at 312.674 83.312 0) (unit 1)
+    (in_bom no) (on_board yes) (dnp no) (fields_autoplaced)
+    (property "Reference" "LOGO3" (at 312.674 76.327 0)
+      (effects (font (size 1.27 1.27)) hide)
+    )
+    (property "Value" "Teacup Logo" (at 320.04 83.312 0)
+      (effects (font (size 1.27 1.27)) (justify left))
+    )
+    (property "Footprint" "teacup:TClogo-med" (at 312.674 83.312 0)
+      (effects (font (size 1.27 1.27)) hide)
+    )
+    (property "Datasheet" "~" (at 312.674 83.312 0)
+      (effects (font (size 1.27 1.27)) hide)
+    )
+    (property "Sim.Enable" "0" (at 312.674 83.312 0)
+      (effects (font (size 1.27 1.27)) hide)
+    )
+    (instances
+      (project "12-30-23-Teacup.kicad_pcb-revC"
+        (path "/6e7ef4e6-2026-4726-8de0-60238113f775"
+          (reference "LOGO3") (unit 1)
+        )
+      )
